File: detector.kicad_pcb (KiCad board)
At the start: 2 copper layers, 43 x 43 mm, 27 parts, among them J1 RF_IN_1, J2 DET_OUT_1, J3 RF_IN_2, J4 DET_OUT_2, P1 4.7k, P2 4.7k

Commit message: Bumping revision to 1.1, put CC license on silk
Other:
- board text added: "Design by Matt Weyland, HB9FRV Rev 1.1, (c) 2019 CC BY-SA 4.0"
- board text removed: "Design by Matt Weyland, HB9FRV Rev 1.0, (c) 2019"
Changed lines of the file:
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@@
     (effects (font (size 1 1) (thickness 0.2)))
   )
-  (gr_text "Design by Matt Weyland, HB9FRV\nRev 1.0, (c) 2019" (at 122.5 66) (layer F.SilkS)
+  (gr_text "Design by Matt Weyland, HB9FRV\nRev 1.1, (c) 2019 CC BY-SA 4.0" (at 122.5 66) (layer F.SilkS)
     (effects (font (size 0.9 0.9) (thickness 0.2)))
   )
